Commit message: Add files via upload

File: urdf/swcr_main.urdf.xacro (robot description, xacro)
@@ -44,4 +44,10 @@
     </collision>
   </link>
+  <link name="base_footprint"/>
+  <joint name="base_footprint_joint" type="fixed">
+    <parent link="base_footprint"/>
+    <child link="base_link"/>
+    <origin xyz="0 0 0.05" rpy="0 0 0"/>
+  </joint>
   <link
     name="clampfr_link">
@@ -182,9 +188,8 @@
     <collision>
       <origin
-        xyz="0 0 0"
-        rpy="0 0 0" />
-      <geometry>
-        <mesh
-          filename="package://swcr_main/meshes/wheelfr_link.STL" />
+        xyz="-0.02 0 0"
+        rpy="0 1.5708 0" />
+      <geometry>
+        <cylinder radius="0.05" length="0.035"/>
       </geometry>
     </collision>
@@ -205,6 +210,5 @@
   <transmission name="wheelfr_trans">
     <type>transmission_interface/SimpleTransmission</type>
-    <actuator name="wheelfr_actuator">
-      <hardwareInterface>VelocityJointInterface</hardwareInterface>
+    <actuator name="$wheelfr_motor">
       <mechanicalReduction>1</mechanicalReduction>
     </actuator>
@@ -213,4 +217,12 @@
     </joint>
   </transmission>
+  <gazebo reference="wheelfr_link">
+      <mu1 value="200.0"/>
+      <mu2 value="100.0"/>
+      <minDepth>0.005</minDepth>
+      <kp value="10000000.0" />
+      <kd value="1.0" />
+    <material>Gazebo/Grey</material>
+   </gazebo>
   <link
     name="clampfl_link">
@@ -351,9 +363,8 @@
     <collision>
       <origin
-        xyz="0 0 0"
-        rpy="0 0 0" />
-      <geometry>
-        <mesh
-          filename="package://swcr_main/meshes/wheelfl_link.STL" />
+        xyz="-0.02 0 0"
+        rpy="0 1.5708 0" />
+      <geometry>
+        <cylinder radius="0.05" length="0.035"/>
       </geometry>
     </collision>
@@ -374,6 +385,5 @@
   <transmission name="wheelfl_trans">
     <type>transmission_interface/SimpleTransmission</type>
-    <actuator name="wheelfl_actuator">
-      <hardwareInterface>VelocityJointInterface</hardwareInterface>
+    <actuator name="$wheelfl_motor">
       <mechanicalReduction>1</mechanicalReduction>
     </actuator>
@@ -382,4 +392,12 @@
     </joint>
   </transmission>
+  <gazebo reference="wheelfl_link">
+      <mu1 value="200.0"/>
+      <mu2 value="100.0"/>
+      <minDepth>0.005</minDepth>
+      <kp value="10000000.0" />
+      <kd value="1.0" />
+    <material>Gazebo/Grey</material>
+   </gazebo>
   <link
     name="clampbl_link">
@@ -520,9 +538,8 @@
     <collision>
       <origin
-        xyz="0 0 0"
-        rpy="0 0 0" />
-      <geometry>
-        <mesh
-          filename="package://swcr_main/meshes/wheelbl_link.STL" />
+        xyz="-0.02 0 0"
+        rpy="0 1.5708 0" />
+      <geometry>
+        <cylinder radius="0.05" length="0.035"/>
       </geometry>
     </collision>
@@ -540,9 +557,22 @@
     <axis
       xyz="1 0 0" />
-    <mimic
-      joint="wheelfl_joint"
-      multiplier="1"
-      offset="0" />
-  </joint>
+  </joint>
+  <transmission name="wheelbl_trans">
+    <type>transmission_interface/SimpleTransmission</type>
+    <actuator name="$wheelbl_motor">
+      <mechanicalReduction>1</mechanicalReduction>
+    </actuator>
+    <joint name="wheelbl_joint">
+      <hardwareInterface>hardware_interface/VelocityJointInterface</hardwareInterface>
+    </joint>
+  </transmission>
+  <gazebo reference="wheelbl_link">
+       <mu1 value="200.0"/>
+       <mu2 value="100.0"/>
+       <minDepth>0.005</minDepth>
+      <kp value="10000000.0" />
+      <kd value="1.0" />
+    <material>Gazebo/Grey</material>
+   </gazebo>
   <link
     name="clampbr_link">
@@ -683,9 +713,8 @@
     <collision>
       <origin
-        xyz="0 0 0"
-        rpy="0 0 0" />
-      <geometry>
-        <mesh
-          filename="package://swcr_main/meshes/wheelbr_link.STL" />
+      xyz="-0.02 0 0"
+      rpy="0 1.5708 0" />
+      <geometry>
+        <cylinder radius="0.05" length="0.035"/>
       </geometry>
     </collision>
@@ -703,9 +732,22 @@
     <axis
       xyz="1 0 0" />
-    <mimic
-      joint="wheelfr_joint"
-      multiplier="1"
-      offset="0" />
-  </joint>
+  </joint>
+  <transmission name="wheelbr_trans">
+    <type>transmission_interface/SimpleTransmission</type>
+    <actuator name="$wheelbr_motor">
+      <mechanicalReduction>1</mechanicalReduction>
+    </actuator>
+    <joint name="wheelbr_joint">
+      <hardwareInterface>hardware_interface/VelocityJointInterface</hardwareInterface>
+    </joint>
+  </transmission>
+  <gazebo reference="wheelbr_link">
+      <mu1 value="200.0"/>
+      <mu2 value="100.0"/>
+      <minDepth>0.005</minDepth>
+      <kp value="10000000.0" />
+      <kd value="1.0" />
+    <material>Gazebo/Grey</material>
+   </gazebo>
   <link
     name="bin_link">
@@ -803,5 +845,5 @@
   <joint
     name="pan_joint"
-    type="continuous">
+    type="revolute">
     <origin
       xyz="0.12 0 0.0075"
@@ -814,21 +856,23 @@
       xyz="0 0 1" />
     <limit
+      lower="0"
+      upper ="1.57"
       effort="30"
       velocity="0.5" />
   </joint>
-  <transmission name="pan_trans">
-    <type>transmission_interface/SimpleTransmission</type>
-    <actuator name="pan_actuator">
-      <hardwareInterface>EffortJointInterface</hardwareInterface>
-      <mechanicalReduction>1</mechanicalReduction>
-    </actuator>
-    <joint name="pan_joint">
-      <hardwareInterface>hardware_interface/EffortJointInterface</hardwareInterface>
-    </joint>
-  </transmission>
   <gazebo>
     <plugin name="gazebo_ros_control" filename="libgazebo_ros_control.so">
-      <robotNamespace>/swcr</robotNamespace>
+      <robotNamespace>/</robotNamespace>
+      <robotSimType>gazebo_ros_control/DefaultRobotHWSim</robotSimType>
+      <legacyModeNS>true</legacyModeNS>
     </plugin>
   </gazebo>
+      <gazebo>
+        <plugin name="gazebo_ros_p3d" filename="libgazebo_ros_p3d.so">
+            <updateRate>100</updateRate>
+            <bodyName>base_footprint</bodyName>
+            <topicName>exact_pose</topicName>
+            <frameName>map</frameName>
+        </plugin>
+    </gazebo>
 </robot>

Commit message: Add files via upload

File: urdf/swcr_main.urdf.xacro (robot description, xacro)
@@ -218,9 +218,6 @@
   </transmission>
   <gazebo reference="wheelfr_link">
-      <mu1 value="200.0"/>
-      <mu2 value="100.0"/>
-      <minDepth>0.005</minDepth>
       <kp value="10000000.0" />
-      <kd value="1.0" />
+      <kd value="1"/>
     <material>Gazebo/Grey</material>
    </gazebo>
@@ -374,6 +371,6 @@
     type="continuous">
     <origin
-      xyz="0 0.007 0.0343"
-      rpy="0.80263 1.5708 0" />
+      xyz="0 0.007 0.0686"
+      rpy="0 -1.5708 0" />
     <parent
       link="motorfl_link" />
@@ -393,9 +390,6 @@
   </transmission>
   <gazebo reference="wheelfl_link">
-      <mu1 value="200.0"/>
-      <mu2 value="100.0"/>
-      <minDepth>0.005</minDepth>
       <kp value="10000000.0" />
-      <kd value="1.0" />
+      <kd value="1"/>
     <material>Gazebo/Grey</material>
    </gazebo>
@@ -549,6 +543,6 @@
     type="continuous">
     <origin
-      xyz="0 0.007 0.0343"
-      rpy="0.80263 1.5708 0" />
+      xyz="0 0.007 0.0686"
+      rpy="0 -1.5708 0" />
     <parent
       link="motorbl_link" />
@@ -568,9 +562,6 @@
   </transmission>
   <gazebo reference="wheelbl_link">
-       <mu1 value="200.0"/>
-       <mu2 value="100.0"/>
-       <minDepth>0.005</minDepth>
       <kp value="10000000.0" />
-      <kd value="1.0" />
+      <kd value="1"/>
     <material>Gazebo/Grey</material>
    </gazebo>
@@ -725,5 +716,5 @@
     <origin
       xyz="0 0.007 0.0343"
-      rpy="0.29376 1.5708 0" />
+      rpy="0 1.5708 0" />
     <parent
       link="motorbr_link" />
@@ -743,9 +734,6 @@
   </transmission>
   <gazebo reference="wheelbr_link">
-      <mu1 value="200.0"/>
-      <mu2 value="100.0"/>
-      <minDepth>0.005</minDepth>
       <kp value="10000000.0" />
-      <kd value="1.0" />
+      <kd value="1"/>
     <material>Gazebo/Grey</material>
    </gazebo>
@@ -810,12 +798,12 @@
         rpy="0 0 0" />
       <mass
-        value="0" />
-      <inertia
-        ixx="0"
-        ixy="0"
-        ixz="0"
-        iyy="0"
-        iyz="0"
-        izz="0" />
+        value="1" />
+      <inertia
+        ixx="1"
+        ixy="1"
+        ixz="1"
+        iyy="1"
+        iyz="1"
+        izz="1" />
     </inertial>
     <visual>
@@ -861,4 +849,13 @@
       velocity="0.5" />
   </joint>
+    <transmission name="pan_trans">
+    <type>transmission_interface/SimpleTransmission</type>
+    <actuator name="$pan_motor">
+      <mechanicalReduction>1</mechanicalReduction>
+    </actuator>
+    <joint name="pan_joint">
+      <hardwareInterface>hardware_interface/EffortJointInterface</hardwareInterface>
+    </joint>
+</transmission>
   <gazebo>
     <plugin name="gazebo_ros_control" filename="libgazebo_ros_control.so">
